Commit message: space_station_gnc is removed

File: urdf/ISS_stationaryFromNasa.urdf (robot description, URDF)
Before this commit: robot ISS_stationaryFromNasa, 1 links, 0 joints
Links:
- link Root: geometry visual mesh filename=package://demo_nauka_incident2021_estimate/urdf/meshes/AMS2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 scale=1. 1. 1.; visual mesh filename=package://demo_nauka_incident2021_estimate/urdf/meshes/Cube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 scale=1. 1. 1.
